Commit message: Updated robot.acro with working skid steer

File: src/enph353_ros_lab/urdf/robot.xacro (robot description, xacro)
@@ -1,12 +1,11 @@
 <?xml version='1.0'?>
-<robot name="bot" xmlns:xacro="http://www.ros.org/wiki/xacro">
+<robot name="robot" xmlns:xacro="http://www.ros.org/wiki/xacro">
   <xacro:property name="chassis_width" value="0.15"/>
   <xacro:property name="chassis_length" value="0.2"/>
   <xacro:property name="chassis_height" value="0.05"/>
-  <xacro:property name="chassis_mass" value="0.5"/>
+  <xacro:property name="chassis_mass" value=".5"/>
   <xacro:property name="wheel_radius" value="0.04"/>
   <xacro:property name="wheel_width" value="0.03"/>
-  <xacro:property name="wheel_mass" value="0.1"/>
-  <!-- <xacro:include filename="$(find enph353_ros_lab)/urdf/robot.gazebo" /> -->
+ <xacro:property name="camera_link" value="0.05" /> <!-- Size of square 'camera' box -->
   <xacro:include filename="$(find enph353_ros_lab)/urdf/macros.xacro" />
   <link name='chassis'>
@@ -18,179 +17,184 @@
     </collision>
     <visual name='chassis_visual'>
+      <origin xyz="0 0 0" rpy=" 0 0 0"/>
+      <geometry>
+        <box size="${chassis_length} ${chassis_width} ${chassis_height}"/>
+      </geometry>
+      <surface>
+        <friction>
+          <ode>
+            <mu>0.1</mu>
+            <mu2>0.1</mu2>
+          </ode>
+        </friction>
+      </surface>
+    </visual>
+  </link>
+<link name='wheel1'>
+	<xacro:cylinder_inertial name="wheel1" m=".01" r ="${wheel_radius}" h="${wheel_width}" />
+   <collision name='wheel1'>
+      <geometry>
+        <cylinder length="${wheel_width}" radius="${wheel_radius}"/>
+      </geometry>
+      <surface>
+        <friction>
+          <ode>
+            <mu>.1</mu>
+            <mu2>.1</mu2>
+          </ode>
+        </friction>
+      </surface>
+<origin rpy="1.57075 0 0" xyz="0 0 0"/>
+    </collision>
+   <visual>
+      <origin rpy="1.57075 0 0" xyz="0 0 0"/>
+      <geometry>
+        <cylinder length="${wheel_width}" radius="${wheel_radius}"/>
+      </geometry>
+    </visual>
+</link>
+<link name='wheel2'>
+	<xacro:cylinder_inertial name="wheel2" m=".01" r ="${wheel_radius}" h="${wheel_width}" />
+   <collision name='wheel1'>
+      <geometry>
+        <cylinder length="${wheel_width}" radius="${wheel_radius}"/>
+      </geometry>
+      <surface>
+        <friction>
+          <ode>
+            <mu>.1</mu>
+            <mu2>.1</mu2>
+          </ode>
+        </friction>
+      </surface>
+    </collision>
+   <visual>
+      <origin rpy="1.57075 0 0" xyz="0 0 0"/>
+      <geometry>
+        <cylinder length="${wheel_width}" radius="${wheel_radius}"/>
+      </geometry>
+<origin rpy="1.57075 0 0" xyz="0 0 0"/>
+    </visual>
+</link>
+<link name='wheel3'>
+	<xacro:cylinder_inertial name="wheel3" m=".01" r ="${wheel_radius}" h="${wheel_width}" />
+   <collision name='wheel1'>
+      <geometry>
+        <cylinder length="${wheel_width}" radius="${wheel_radius}"/>
+      </geometry>
+      <surface>
+        <friction>
+          <ode>
+            <mu>.1</mu>
+            <mu2>.1</mu2>
+          </ode>
+        </friction>
+      </surface>
+<origin rpy="1.57075 0 0" xyz="0 0 0"/>
+    </collision>
+   <visual>
+      <origin rpy="1.57075 0 0" xyz="0 0 0"/>
+      <geometry>
+        <cylinder length="${wheel_width}" radius="${wheel_radius}"/>
+      </geometry>
+<origin rpy="1.57075 0 0" xyz="0 0 0"/>
+    </visual>
+</link>
+<link name='wheel4'>
+	<xacro:cylinder_inertial name="wheel1" m=".01" r ="${wheel_radius}" h="${wheel_width}" />
+   <collision name='wheel4'>
+      <geometry>
+        <cylinder length="${wheel_width}" radius="${wheel_radius}"/>
+      </geometry>
+      <surface>
+        <friction>
+          <ode>
+            <mu>.1</mu>
+            <mu2>.1</mu2>
+          </ode>
+        </friction>
+      </surface>
+<origin rpy="1.57075 0 0" xyz="0 0 0"/>
+    </collision>
+   <visual>
+      <origin rpy="1.57075 0 0" xyz="0 0 0"/>
+      <geometry>
+        <cylinder length="${wheel_width}" radius="${wheel_radius}"/>
+      </geometry>
+    </visual>
+</link>
+  <joint name="joint1" type="continuous">
+<axis xyz=" 0 1 0"/>
+    <parent link="chassis"/>
+    <child link="wheel1"/>
+    <origin xyz=".1 .09 0" rpy="0 0 0" />
+  </joint>
+  <joint name="joint2" type="continuous">
+<axis xyz=" 0 1 0"/>
+    <parent link="chassis"/>
+    <child link="wheel2"/>
+    <origin xyz="-.1 .09 0" rpy="0 0 0" />
+  </joint>
+  <joint name="joint3" type="continuous">
+<axis xyz=" 0 1 0"/>
+    <parent link="chassis"/>
+    <child link="wheel3"/>
+    <origin xyz=".1 -.09 0" rpy="0 0 0" />
+  </joint>
+  <joint name="joint4" type="continuous">
+    <axis xyz=" 0 1 0"/>
+    <parent link="chassis"/>
+    <child link="wheel4"/>
+    <origin xyz="-.1 -.09 0" rpy="0 0 0" />
+  </joint>
+<gazebo>
+  <plugin name="skid_steer_drive_controller" filename="libgazebo_ros_skid_steer_drive.so">
+    <updateRate>100.0</updateRate>
+    <robotNamespace>/</robotNamespace>
+    <leftFrontJoint>joint1</leftFrontJoint>
+    <rightFrontJoint>joint3</rightFrontJoint>
+    <leftRearJoint>joint2</leftRearJoint>
+    <rightRearJoint>joint4</rightRearJoint>
+    <wheelSeparation>.18</wheelSeparation>
+    <wheelDiameter>0.08</wheelDiameter>
+    <robotBaseFrame>base_link</robotBaseFrame>
+    <torque>20</torque>
+    <topicName>cmd_vel</topicName>
+    <broadcastTF>false</broadcastTF>
+  </plugin>
+</gazebo>
+<joint name="camera_joint" type="fixed">
+    <axis xyz="0 1 0" />
+    <origin xyz=".1 0 .05" rpy="0 0.5 0"/>
+    <parent link="chassis"/>
+    <child link="camera_link"/>
+  </joint>
+  <!-- Camera -->
+  <link name="camera_link">
+    <collision>
       <origin xyz="0 0 0" rpy="0 0 0"/>
       <geometry>
-        <box size="${chassis_length} ${chassis_width} ${chassis_height}"/>
-      </geometry>
-    </visual>
+    <box size="${camera_link} ${camera_link} ${camera_link}"/>
+      </geometry>
+    </collision>
+    <visual>
+      <origin xyz="0 0 0" rpy="0 0 0"/>
+      <geometry>
+    <box size="${camera_link} ${camera_link} ${camera_link}"/>
+      </geometry>
+      <material name="red"/>
+    </visual>
+    <inertial>
+      <mass value="1e-5" />
+      <origin xyz="0 0 0" rpy="0 0 0"/>
+      <inertia ixx="1e-6" ixy="0" ixz="0" iyy="1e-6" iyz="0" izz="1e-6" />
+    </inertial>
   </link>
-  <link name='wheelBL'>
-  <xacro:cylinder_inertial name='wheelBL' m='${wheel_mass}' r='${wheel_radius}' h='${wheel_width}'/>
-    <collision name='wheelBL_collision'>
-      <origin xyz="0 0 0" rpy="1.57 0 0"/>
-      <geometry>
-        <cylinder radius='${wheel_radius}' length='${wheel_width}'/>
-      </geometry>
-    </collision>
-    <visual name='wheelBL_visual'>
-      <origin xyz='0 0 0' rpy='1.57 0 0'/>
-      <geometry>
-        <cylinder radius='${wheel_radius}' length='${wheel_width}'/>
-      </geometry>
-      <surface>
-        <friction>
-          <ode>
-	    			<mu>1</mu>
-            <mu2>1</mu2>
-	    			<slip1>1.0</slip1>
-            <slip2>1.0</slip2>
-	 			  </ode>
-        </friction>
-      </surface>
-    </visual>
-  </link>
-  <link name='wheelBR'>
-  <xacro:cylinder_inertial name='wheelBR' m='${wheel_mass}' r='${wheel_radius}' h='${wheel_width}'/>
-    <collision name='wheelBR_collision'>
-      <origin xyz="0 0 0" rpy="1.57 0 0"/>
-      <geometry>
-        <cylinder radius='${wheel_radius}' length='${wheel_width}'/>
-      </geometry>
-    </collision>
-    <visual name='wheelBR_visual'>
-      <origin xyz='0 0 0' rpy='1.57 0 0'/>
-      <geometry>
-        <cylinder radius='${wheel_radius}' length='${wheel_width}'/>
-      </geometry>
-      <surface>
-        <friction>
-          <ode>
-	    			<mu>1</mu>
-          	<mu2>1</mu2>
-	    			<slip1>1.0</slip1>
-          	<slip2>1.0</slip2>
-	  			</ode>
-        </friction>
-      </surface>
-    </visual>
-  </link>
-  <link name='wheelFL'>
-  <xacro:cylinder_inertial name='wheelFL' m='${wheel_mass}' r='${wheel_radius}' h='${wheel_width}'/>
-    <collision name='wheelFL_collision'>
-      <origin xyz="0 0 0" rpy="1.57 0 0"/>
-      <geometry>
-        <cylinder radius='${wheel_radius}' length='${wheel_width}'/>
-      </geometry>
-      <surface>
-        <friction>
-          <ode>
-	    			<mu>1</mu>
-            <mu2>1</mu2>
-	    			<slip1>1.0</slip1>
-            <slip2>1.0</slip2>
-	  			</ode>
-        </friction>
-      </surface>
-    </collision>
-    <visual name='wheelFL_visual'>
-      <origin xyz='0 0 0' rpy='1.57 0 0'/>
-      <geometry>
-        <cylinder radius='${wheel_radius}' length='${wheel_width}'/>
-      </geometry>
-    </visual>
-  </link>
-  <link name='wheelFR'>
-  <xacro:cylinder_inertial name='wheelFR' m='${wheel_mass}' r='${wheel_radius}' h='${wheel_width}'/>
-    <collision name='wheelFR_collision'>
-      <origin xyz="0 0 0" rpy="1.57 0 0"/>
-      <geometry>
-        <cylinder radius='${wheel_radius}' length='${wheel_width}'/>
-      </geometry>
-      <surface>
-        <friction>
-          <ode>
-	    			<mu>1</mu>
-            <mu2>1</mu2>
-	    			<slip1>1.0</slip1>
-            <slip2>1.0</slip2>
-	 			  </ode>
-        </friction>
-      </surface>
-    </collision>
-    <visual name='wheelFR_visual'>
-      <origin xyz='0 0 0' rpy='1.57 0 0'/>
-      <geometry>
-        <cylinder radius='${wheel_radius}' length='${wheel_width}'/>
-      </geometry>
-    </visual>
-  </link>
-  <link name='camera_mount'>
-    <inertial>
-      <mass value='1e-5'/>
-      <origin xyz='0 0 0' rpy='0 0 0'/>
-      <inertia ixx='1e-6' ixy='0' ixz='0' iyy='1e-6' iyz='0' izz='1e-6'/>
-    </inertial>
-    <collision>
-      <origin xyz='0 0 0' rpy='0 0 0'/>
-      <geometry>
-        <box size='0.05 0.05 0.05'/>
-      </geometry>
-    </collision>
-    <visual>
-      <origin xyz='0 0 0' rpy='0 0 0'/>
-      <geometry>
-        <box size='0.05 0.05 0.05'/>
-      </geometry>
-    </visual>
-  </link>
-  <joint name='axleBL' type='continuous'>
-    <origin xyz='${-chassis_length/2} ${(chassis_width+wheel_width)/2} 0'/>
-    <parent link='chassis'/>
-    <child link='wheelBL'/>
-    <axis xyz='0 1 0'/>
-  </joint>
-  <joint name='axleBR' type='continuous'>
-    <origin xyz='${-chassis_length/2} ${-(chassis_width+wheel_width)/2} 0'/>
-    <parent link='chassis'/>
-    <child link='wheelBR'/>
-    <axis xyz='0 1 0'/>
-  </joint>
-  <joint name='axleFL' type='continuous'>
-    <origin xyz='${chassis_length/2} ${(chassis_width+wheel_width)/2} 0'/>
-    <parent link='chassis'/>
-    <child link='wheelFL'/>
-    <axis xyz='0 1 0'/>
-  </joint>
-  <joint name='axleFR' type='continuous'>
-    <origin xyz='${chassis_length/2} ${-(chassis_width+wheel_width)/2} 0'/>
-    <parent link='chassis'/>
-    <child link='wheelFR'/>
-    <axis xyz='0 1 0'/>
-  </joint>
-  <joint name='camera_joint' type='fixed'>
-    <origin xyz='${chassis_length/2} 0 0'/>
-    <parent link='chassis'/>
-    <child link='camera_mount'/>
-    <axis xyz='0 1 0'/>
-  </joint>
-  <gazebo>
-    <plugin name='skid_steer_drive_controller' filename='libgazebo_ros_skid_steer_drive.so'>
-      <updateRate>100</updateRate>
-      <robotNamespace>/</robotNamespace>
-			<leftFrontJoint>axleFL</leftFrontJoint>
-      <rightFrontJoint>axleFR</rightFrontJoint>
-      <leftRearJoint>axleBL</leftRearJoint>
-      <rightRearJoint>axleBR</rightRearJoint>
-      <wheelSeparation>${chassis_width+wheel_width)</wheelSeparation>
-      <wheelDiameter>${2*wheel_radius}</wheelDiameter>
-			<robotBaseFrame>chassis</robotBaseFrame>
-      <torque>20</torque>
-      <topicName>cmd_vel</topicName>
-    </plugin>
-  </gazebo>
-  <gazebo reference='camera_mount'>
-    <sensor type='camera' name='camera1'>
+ <!-- camera -->
+  <gazebo reference="camera_link">
+    <sensor type="camera" name="camera1">
       <update_rate>30.0</update_rate>
-      <camera name='head'>
-        <horizontal_fov>1.4</horizontal_fov>
+      <camera name="head">
+        <horizontal_fov>1.3962634</horizontal_fov>
         <image>
           <width>800</width>
@@ -204,15 +208,18 @@
         <noise>
           <type>gaussian</type>
+          <!-- Noise is sampled independently per pixel on each frame.
+               That pixel's noise value is added to each of its color
+               channels, which at that point lie in the range [0,1]. -->
           <mean>0.0</mean>
           <stddev>0.007</stddev>
         </noise>
       </camera>
-      <plugin name='camera_controller' filename='libgazebo_ros_camera.so'>
+      <plugin name="camera_controller" filename="libgazebo_ros_camera.so">
         <alwaysOn>true</alwaysOn>
         <updateRate>0.0</updateRate>
-        <cameraName>bot/camera1</cameraName>
+        <cameraName>rrbot/camera1</cameraName>
         <imageTopicName>image_raw</imageTopicName>
         <cameraInfoTopicName>camera_info</cameraInfoTopicName>
-        <frameName>camera_mount</frameName>
+        <frameName>camera_link</frameName>
         <hackBaseline>0.07</hackBaseline>
         <distortionK1>0.0</distortionK1>
