Commit message: Added baby

File: src/2019F_competition_students/adeept_awr/adeept_awr_description/urdf/adeept_awr.urdf (robot description, URDF)
Before this commit: robot adeept_awr, 7 links, 6 joints
Links:
- link battery: geometry collision box size=0.145 0.065 0.015
- link camera_link: geometry collision box size=1e-6 1e-6 1e-6
- link chassis: geometry collision box size=0.13 0.12 0.08; visual mesh filename=package://adeept_awr_description/baby.obj scale=0.01 0.01 0.01
- link front_left_wheel: geometry collision cylinder length=0.025 radius=0.0325
- link front_right_wheel: geometry collision cylinder length=0.025 radius=0.0325
- link rear_left_wheel: geometry collision cylinder length=0.025 radius=0.0325
- link rear_right_wheel: geometry collision cylinder length=0.025 radius=0.0325
